Commit message: [config,user] update setting and models

File: user/kxr_uav/rleg.urdf (robot description, URDF)
Before this commit: robot rleg, 7 links, 6 joints
Links:
- link LINK5: geometry collision mesh filename=package://robot_assembler/meshes/kxr_uav/wheel_foot.STL scale=0.001000 0.001000 0.001000; visual mesh filename=package://robot_assembler/meshes/kxr_uav/wheel_foot.STL scale=0.001000 0.001000 0.001000
Joints:
- joint JOINT3: origin xyz=-0.023500 -0.053000 -0.000500 rpy=-0.00000000 -0.00000000 1.57079633 -> xyz=-0.023500 -0.053000 -0.000500 rpy=0.00000000 -0.00000000 1.57079633
- joint JOINT5: origin xyz=0.065000 -0.000000 0.017000 rpy=0.65131141 -1.57079633 2.49028124 -> xyz=0.065000 -0.000000 0.017000 rpy=0.89880790 -1.57079633 2.24278475

File: user/kxr_uav/torso.urdf (robot description, URDF)
Before this commit: robot torso, 3 links, 2 joints
Links:
- link BASE: mass 0.402166 -> 0.485674; geometry collision mesh filename=package://robot_assembler/meshes/kxr_uav/uav_backpack.STL scale=0.001000 0.001000 0.001000; collision mesh filename=package://robot_assembler/meshes/kxr_uav/uav_backpack_mount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 scale=0.001000 0.001000 0.001000
Joints:
- joint JOINT1: origin xyz=-0.000000 -0.018000 0.032500 rpy=1.42371797 -1.57079633 0.14707836 -> xyz=-0.000000 -0.018000 0.032500 rpy=1.78188966 -1.57079633 -0.21109333
