Commit message: [user] add fullbody models

File: user/kxr_uav/torso.urdf (robot description, URDF)
Before this commit: robot torso, 3 links, 2 joints
Links:
- link BASE: mass 0.485674 -> 0.538474; geometry collision mesh filename=package://robot_assembler/meshes/kxr_uav/uav_backpack.STL scale=0.001000 0.001000 0.001000; collision mesh filename=package://robot_assembler/meshes/kxr_uav/uav_backpack_mount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 scale=0.001000 0.001000 0.001000
