Commit message: [user] update rarm roboasm

File: user/kxr_uav/rarm.urdf (robot description, URDF)
Before this commit: robot rarm, 8 links, 7 joints
Links:
- added link LINK7, mass 0.013908; collision mesh filename=package://robot_assembler/meshes/mesh_FINGER.dae scale=1.000000 1.000000 1.000000; visual mesh filename=package://robot_assembler/meshes/mesh_FINGER.dae scale=1.000000 1.000000 1.000000
Joints:
- added joint JOINT7: type revolute, parent LINK5, child LINK7, origin xyz=-0.071768 -0.000734 0.000500 rpy=-0.00000000 0.00000000 1.43420534, axis 0 0 1, limit lower=-3.14159 upper=3.14159 effort=200 velocity=40
- joint JOINT2: origin xyz=-0.017500 0.058000 -0.017500 rpy=1.57079633 -0.00000000 -1.57079633 -> xyz=-0.021417 0.056671 -0.017500 rpy=1.57079633 -0.00000000 -1.50250083
- joint JOINT3: origin xyz=-0.070000 -0.000000 -0.018000 rpy=-1.36194019 1.57079633 1.77965246 -> xyz=-0.070000 -0.000000 -0.018000 rpy=-1.36238365 1.57079633 1.77920900
- joint JOINT4: origin xyz=-0.017000 0.000000 0.027500 rpy=-3.14159265 1.57079633 -3.14159265 -> xyz=-0.017000 0.000000 0.027500 rpy=3.14159265 1.57079633 -3.14159265
- joint JOINT6: origin xyz=-0.060500 0.010500 0.000500 rpy=-0.00000000 0.00000000 1.57079633 -> xyz=-0.058507 0.018640 0.000500 rpy=-0.00000000 0.00000000 1.43420534
