Commit message: [user] update leg model

File: user/kxr_uav/kxr_uav_fullbody.urdf (robot description, URDF)
Before this commit: robot kxr_uav_fullbody, 39 links, 38 joints
Links:
- link LINK26: mass 0.026432 -> 0.025166; geometry collision mesh filename=package://robot_assembler/meshes/mesh_BOTTOM-ARM20.dae scale=1.000000 1.000000 1.000000; collision mesh filename=package://robot_assembler/meshes/mesh_BOTTOM-ARM38.dae scale=1.000000 1.000000 1.000000
- link LINK33: mass 0.026432 -> 0.025166; geometry collision mesh filename=package://robot_assembler/meshes/mesh_BOTTOM-ARM20.dae scale=1.000000 1.000000 1.000000; collision mesh filename=package://robot_assembler/meshes/mesh_BOTTOM-ARM38.dae scale=1.000000 1.000000 1.000000
Joints:
- joint JOINT27: origin xyz=-0.064000 -0.000000 -0.000000 rpy=-0.00000000 -0.00000000 0.00000000 -> xyz=-0.058000 -0.000000 -0.000000 rpy=0.00000000 -0.00000000 -1.04719755
- joint JOINT28: origin xyz=-0.023500 -0.053000 -0.000500 rpy=-0.00000000 -0.00000000 1.57079633 -> xyz=-0.023500 -0.053000 -0.000500 rpy=-0.00000000 -0.00000000 1.04719755
- joint JOINT30: origin xyz=0.065000 -0.000000 0.017000 rpy=1.07262664 -1.57079633 2.06896601 -> xyz=0.065000 -0.000000 0.017000 rpy=1.04666457 -1.57079633 2.09492808
- joint JOINT34: origin xyz=-0.064000 -0.000000 -0.000000 rpy=-0.00000000 -0.00000000 0.00000000 -> xyz=-0.058000 -0.000000 -0.000000 rpy=0.00000000 -0.00000000 -1.04719755
- joint JOINT35: origin xyz=-0.023500 -0.053000 -0.000500 rpy=-0.00000000 -0.00000000 1.57079633 -> xyz=-0.023500 -0.053000 -0.000500 rpy=-0.00000000 -0.00000000 1.04719755
- joint JOINT37: origin xyz=0.065000 -0.000000 0.017000 rpy=0.90821104 -1.57079633 2.23338162 -> xyz=0.065000 -0.000000 0.017000 rpy=1.19112612 -1.57079633 1.95046654

Commit message: [user] update model files

File: user/kxr_uav/kxr_uav_fullbody.urdf (robot description, URDF)
Before this commit: robot kxr_uav_fullbody, 39 links, 38 joints
Links:
- added link LINK38, mass 0.045736; collision mesh filename=package://robot_assembler/meshes/mesh_BOTTOM-ARM28.dae scale=1.000000 1.000000 1.000000; collision mesh filename=package://robot_assembler/meshes/mesh_BOTTOM-SPACER.dae scale=1.000000 1.000000 1.000000
- added link LINK39, mass 0.03987; collision mesh filename=package://robot_assembler/meshes/kxr_uav/wheel_foot.STL scale=0.001000 0.001000 0.001000; visual mesh filename=package://robot_assembler/meshes/kxr_uav/wheel_foot.STL scale=0.001000 0.001000 0.001000
- link LINK14: mass 0.012371 -> 0.013908; geometry collision mesh filename=package://robot_assembler/meshes/mesh_FINGER.dae scale=1.000000 1.000000 1.000000; visual mesh filename=package://robot_assembler/meshes/mesh_FINGER.dae scale=1.000000 1.000000 1.000000
- link LINK15: mass 0.061777 -> 0.012371; geometry collision mesh filename=package://robot_assembler/meshes/mesh_BOTTOM-ARM28.dae scale=1.000000 1.000000 1.000000; collision mesh filename=package://robot_assembler/meshes/mesh_JOINT-BASE.dae scale=1.000000 1.000000 1.000000
- link LINK16: mass 0.021241 -> 0.061777; geometry collision mesh filename=package://robot_assembler/meshes/mesh_CROSS-SERVO-FRAME-A.d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 scale=1.000000 1.000000 1.000000; collision mesh filename=package://robot_assembler/meshes/mesh_CROSS-SERVO-FRAME-B.d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 scale=1.000000 1.000000 1.000000
- link LINK17: mass 0.068898 -> 0.021241; geometry collision mesh filename=package://robot_assembler/meshes/mesh_BOTTOM-ARM26.dae scale=1.000000 1.000000 1.000000; collision mesh filename=package://robot_assembler/meshes/mesh_BOTTOM-ARM38.dae scale=1.000000 1.000000 1.000000
- link LINK18: mass 0.012371 -> 0.068898; geometry collision mesh filename=package://robot_assembler/meshes/mesh_BOTTOM-SPACER.dae scale=1.000000 1.000000 1.000000; collision mesh filename=package://robot_assembler/meshes/mesh_JOINT-BASE.dae scale=1.000000 1.000000 1.000000
- link LINK19: mass 0.061777 -> 0.012371; geometry collision mesh filename=package://robot_assembler/meshes/mesh_BOTTOM-ARM28.dae scale=1.000000 1.000000 1.000000; collision mesh filename=package://robot_assembler/meshes/mesh_JOINT-BASE.dae scale=1.000000 1.000000 1.000000
- link LINK20: mass 0.050016 -> 0.061777; geometry collision mesh filename=package://robot_assembler/meshes/mesh_CROSS-SERVO-FRAME-A.d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 scale=1.000000 1.000000 1.000000; collision mesh filename=package://robot_assembler/meshes/mesh_CROSS-SERVO-FRAME-B.d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 scale=1.000000 1.000000 1.000000
- link LINK21: mass 0.013908 -> 0.050016; geometry collision mesh filename=package://robot_assembler/meshes/mesh_BOTTOM-ARM38.dae scale=1.000000 1.000000 1.000000; collision mesh filename=package://robot_assembler/meshes/mesh_JOINT-BASE.dae scale=1.000000 1.000000 1.000000
- link LINK22: mass 0.035533 -> 0.013908; geometry collision mesh filename=package://robot_assembler/meshes/mesh_FINGER.dae scale=1.000000 1.000000 1.000000; visual mesh filename=package://robot_assembler/meshes/mesh_FINGER.dae scale=1.000000 1.000000 1.000000
- link LINK23: mass 0.01216 -> 0.013908; geometry collision mesh filename=package://robot_assembler/meshes/mesh_FINGER.dae scale=1.000000 1.000000 1.000000; visual mesh filename=package://robot_assembler/meshes/mesh_FINGER.dae scale=1.000000 1.000000 1.000000
- link LINK24: mass 0.012371 -> 0.035533; geometry collision mesh filename=package://robot_assembler/meshes/mesh_JOINT-BASE.dae scale=1.000000 1.000000 1.000000; collision mesh filename=package://robot_assembler/meshes/mesh_JOINT-FRAME-A.dae scale=1.000000 1.000000 1.000000
- link LINK25: mass 0.061777 -> 0.01216; geometry collision mesh filename=package://robot_assembler/meshes/mesh_BOTTOM-ARM28.dae scale=1.000000 1.000000 1.000000; collision mesh filename=package://robot_assembler/meshes/mesh_JOINT-BASE.dae scale=1.000000 1.000000 1.000000
- link LINK26: mass 0.025166 -> 0.012371; geometry collision mesh filename=package://robot_assembler/meshes/mesh_BOTTOM-ARM28.dae scale=1.000000 1.000000 1.000000; collision mesh filename=package://robot_assembler/meshes/mesh_JOINT-BASE.dae scale=1.000000 1.000000 1.000000
- link LINK27: mass 0.055048 -> 0.061777; geometry collision mesh filename=package://robot_assembler/meshes/mesh_CROSS-SERVO-FRAME-A.d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 scale=1.000000 1.000000 1.000000; collision mesh filename=package://robot_assembler/meshes/mesh_CROSS-SERVO-FRAME-B.d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 scale=1.000000 1.000000 1.000000
- link LINK28: mass 0.061777 -> 0.025166; geometry collision mesh filename=package://robot_assembler/meshes/mesh_BOTTOM-ARM20.dae scale=1.000000 1.000000 1.000000; collision mesh filename=package://robot_assembler/meshes/mesh_BOTTOM-ARM38.dae scale=1.000000 1.000000 1.000000
- link LINK29: mass 0.045736 -> 0.055048; geometry collision mesh filename=package://robot_assembler/meshes/mesh_ANGLE-BRACKET.dae scale=1.000000 1.000000 1.000000; collision mesh filename=package://robot_assembler/meshes/mesh_ANGLE-BRACKET.dae scale=1.000000 1.000000 1.000000
- link LINK30: mass 0.03987 -> 0.061777; geometry collision mesh filename=package://robot_assembler/meshes/mesh_CROSS-SERVO-FRAME-A.d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 scale=1.000000 1.000000 1.000000; collision mesh filename=package://robot_assembler/meshes/mesh_CROSS-SERVO-FRAME-B.d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 scale=1.000000 1.000000 1.000000
- link LINK31: mass 0.012371 -> 0.045736; geometry collision mesh filename=package://robot_assembler/meshes/mesh_BOTTOM-ARM28.dae scale=1.000000 1.000000 1.000000; collision mesh filename=package://robot_assembler/meshes/mesh_BOTTOM-SPACER.dae scale=1.000000 1.000000 1.000000
- link LINK32: mass 0.061777 -> 0.03987; geometry collision mesh filename=package://robot_assembler/meshes/kxr_uav/wheel_foot.STL scale=0.001000 0.001000 0.001000; visual mesh filename=package://robot_assembler/meshes/kxr_uav/wheel_foot.STL scale=0.001000 0.001000 0.001000
- link LINK33: mass 0.025166 -> 0.012371; geometry collision mesh filename=package://robot_assembler/meshes/mesh_BOTTOM-ARM28.dae scale=1.000000 1.000000 1.000000; collision mesh filename=package://robot_assembler/meshes/mesh_JOINT-BASE.dae scale=1.000000 1.000000 1.000000
- link LINK34: mass 0.055048 -> 0.061777; geometry collision mesh filename=package://robot_assembler/meshes/mesh_CROSS-SERVO-FRAME-A.d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 scale=1.000000 1.000000 1.000000; collision mesh filename=package://robot_assembler/meshes/mesh_CROSS-SERVO-FRAME-B.d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 scale=1.000000 1.000000 1.000000
- link LINK35: mass 0.061777 -> 0.025166; geometry collision mesh filename=package://robot_assembler/meshes/mesh_BOTTOM-ARM20.dae scale=1.000000 1.000000 1.000000; collision mesh filename=package://robot_assembler/meshes/mesh_BOTTOM-ARM38.dae scale=1.000000 1.000000 1.000000
- link LINK36: mass 0.045736 -> 0.055048; geometry collision mesh filename=package://robot_assembler/meshes/mesh_ANGLE-BRACKET.dae scale=1.000000 1.000000 1.000000; collision mesh filename=package://robot_assembler/meshes/mesh_ANGLE-BRACKET.dae scale=1.000000 1.000000 1.000000
- link LINK37: mass 0.03987 -> 0.061777; geometry collision mesh filename=package://robot_assembler/meshes/mesh_CROSS-SERVO-FRAME-A.d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 scale=1.000000 1.000000 1.000000; collision mesh filename=package://robot_assembler/meshes/mesh_CROSS-SERVO-FRAME-B.d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 scale=1.000000 1.000000 1.000000
Joints:
- added joint JOINT38: type revolute, parent LINK37, child LINK38, origin xyz=-0.021000 -0.017000 -0.018000 rpy=1.57079633 0.00000000 -3.14159265, axis 0 0 1, limit lower=-3.14159 upper=3.14159 effort=200 velocity=40
- added joint JOINT39: type revolute, parent LINK38, child LINK39, origin xyz=0.065000 -0.000000 0.017000 rpy=0.71573506 -1.57079633 2.42585760, axis 0 0 1, limit lower=-3.14159 upper=3.14159 effort=200 velocity=40
- joint JOINT10: origin xyz=-0.070000 -0.000000 -0.018000 rpy=-1.20321187 1.57079633 1.93838078 -> xyz=-0.070000 -0.000000 -0.018000 rpy=-1.46795693 1.57079633 1.67363573
- joint JOINT11: origin xyz=-0.017000 0.000000 0.027500 rpy=3.14159265 1.57079633 3.14159265 -> xyz=-0.017000 0.000000 0.027500 rpy=-3.14159265 1.57079633 -3.14159265
- joint JOINT13: origin xyz=-0.060500 0.010500 0.000500 rpy=-0.00000000 0.00000000 1.57079633 -> xyz=-0.058507 0.018640 0.000500 rpy=-0.00000000 0.00000000 1.43420534
- joint JOINT14: origin xyz=0.051000 -0.007250 0.059500 rpy=-1.57079633 0.00000000 -1.57079633 -> xyz=-0.071768 -0.000734 0.000500 rpy=-0.00000000 0.00000000 1.43420534; parent BASE -> LINK12
- joint JOINT15: origin xyz=0.000000 -0.017000 0.027500 rpy=1.12637712 1.57079633 2.69717344 -> xyz=0.051000 -0.007250 0.059500 rpy=-1.57079633 0.00000000 -1.57079633; parent LINK14 -> BASE
- joint JOINT16: origin xyz=0.000000 -0.018000 0.017000 rpy=1.57079633 0.00000000 0.00000000 -> xyz=0.000000 -0.017000 0.027500 rpy=1.12637712 1.57079633 2.69717344
- joint JOINT17: origin xyz=-0.017500 0.058000 -0.017500 rpy=1.57079633 -0.00000000 -1.57079633 -> xyz=0.000000 -0.018000 0.017000 rpy=1.57079633 0.00000000 0.00000000
- joint JOINT18: origin xyz=-0.070000 -0.000000 -0.018000 rpy=-1.28038351 1.57079633 1.86120914 -> xyz=-0.021417 0.056671 -0.017500 rpy=1.57079633 -0.00000000 -1.50250083
- joint JOINT19: origin xyz=-0.017000 0.000000 0.027500 rpy=3.14159265 1.57079633 3.14159265 -> xyz=-0.070000 -0.000000 -0.018000 rpy=-1.51272860 1.57079633 1.62886405
- joint JOINT20: origin xyz=0.000000 -0.018000 0.017000 rpy=1.57079633 0.00000000 0.00000000 -> xyz=-0.017000 0.000000 0.027500 rpy=-3.14159265 1.57079633 -3.14159265
- joint JOINT21: origin xyz=-0.060500 0.010500 0.000500 rpy=-0.00000000 0.00000000 1.57079633 -> xyz=0.000000 -0.018000 0.017000 rpy=1.57079633 0.00000000 0.00000000
- joint JOINT22: origin xyz=0.000000 -0.007250 0.077500 rpy=-0.00000000 0.00000000 -1.57079633 -> xyz=-0.058507 0.018640 0.000500 rpy=-0.00000000 0.00000000 1.43420534; parent BASE -> LINK21
- joint JOINT23: origin xyz=-0.000000 -0.018000 0.032500 rpy=1.78188966 -1.57079633 -0.21109333 -> xyz=-0.071768 -0.000734 0.000500 rpy=-0.00000000 0.00000000 1.43420534; parent LINK22 -> LINK21
- joint JOINT24: origin xyz=0.044500 -0.010500 -0.051000 rpy=3.14159265 0.00000000 0.00000000 -> xyz=0.000000 -0.007250 0.077500 rpy=-0.00000000 0.00000000 -1.57079633
- joint JOINT25: origin xyz=0.000000 0.017000 0.027500 rpy=2.48054948 1.57079633 0.90975316 -> xyz=-0.000000 -0.018000 0.032500 rpy=1.78188966 -1.57079633 -0.21109333
- joint JOINT26: origin xyz=0.000000 -0.018000 0.017000 rpy=1.57079633 0.00000000 0.00000000 -> xyz=0.044500 -0.010500 -0.051000 rpy=3.14159265 0.00000000 0.00000000; parent LINK25 -> BASE
- joint JOINT27: origin xyz=-0.058000 -0.000000 -0.000000 rpy=0.00000000 -0.00000000 -1.04719755 -> xyz=0.000000 0.017000 0.027500 rpy=2.48054948 1.57079633 0.90975316
- joint JOINT28: origin xyz=-0.023500 -0.053000 -0.000500 rpy=-0.00000000 -0.00000000 1.04719755 -> xyz=0.000000 -0.018000 0.017000 rpy=1.57079633 0.00000000 0.00000000
- joint JOINT29: origin xyz=-0.021000 -0.017000 -0.018000 rpy=1.57079633 0.00000000 -3.14159265 -> xyz=-0.057460 -0.007898 -0.000000 rpy=-0.00000000 -0.00000000 0.13659098
- joint JOINT30: origin xyz=0.065000 -0.000000 0.017000 rpy=1.04666457 -1.57079633 2.09492808 -> xyz=-0.023500 -0.053000 -0.000500 rpy=-0.00000000 -0.00000000 1.57079633
- joint JOINT31: origin xyz=-0.044500 -0.010500 -0.051000 rpy=3.14159265 0.00000000 -3.14159265 -> xyz=-0.021000 -0.017000 -0.018000 rpy=1.57079633 0.00000000 -3.14159265; parent BASE -> LINK30
- joint JOINT32: origin xyz=-0.000000 -0.017000 0.027500 rpy=-1.57079633 1.57079633 0.00000000 -> xyz=0.065000 -0.000000 0.017000 rpy=1.14099359 -1.57079633 2.00059907
- joint JOINT33: origin xyz=0.000000 -0.018000 0.017000 rpy=1.57079633 0.00000000 0.00000000 -> xyz=-0.044500 -0.010500 -0.051000 rpy=3.14159265 0.00000000 -3.14159265; parent LINK32 -> BASE
- joint JOINT34: origin xyz=-0.058000 -0.000000 -0.000000 rpy=0.00000000 -0.00000000 -1.04719755 -> xyz=-0.000000 -0.017000 0.027500 rpy=-1.57079633 1.57079633 0.00000000
- joint JOINT35: origin xyz=-0.023500 -0.053000 -0.000500 rpy=-0.00000000 -0.00000000 1.04719755 -> xyz=0.000000 -0.018000 0.017000 rpy=1.57079633 0.00000000 0.00000000
- joint JOINT36: origin xyz=-0.021000 -0.017000 -0.018000 rpy=1.57079633 0.00000000 -3.14159265 -> xyz=-0.057460 -0.007898 -0.000000 rpy=-0.00000000 -0.00000000 0.13659098
- joint JOINT37: origin xyz=0.065000 -0.000000 0.017000 rpy=1.19112612 -1.57079633 1.95046654 -> xyz=-0.023500 -0.053000 -0.000500 rpy=-0.00000000 -0.00000000 1.57079633
- joint JOINT9: origin xyz=-0.017500 0.058000 -0.017500 rpy=1.57079633 -0.00000000 -1.57079633 -> xyz=-0.021417 0.056671 -0.017500 rpy=1.57079633 -0.00000000 -1.50250083

Commit message: [config,user] changed mass parametors and fixed user file

File: user/kxr_uav/kxr_uav_fullbody.urdf (robot description, URDF)
Before this commit: robot kxr_uav_fullbody, 41 links, 40 joints
Links:
- link BASE: mass 0.538474 -> 0.802232
