Commit message: [user] update actuator name

File: sample/kxr_auv/kxr_auv_fullbody.urdf (robot description, URDF)
Before this commit: robot kxr_auv_fullbody, 25 links, 24 joints
Joints:
- removed joint JOINT0
- removed joint JOINT1
- removed joint JOINT10
- removed joint JOINT11
- removed joint JOINT12
- removed joint JOINT13
- removed joint JOINT14
- removed joint JOINT15
- removed joint JOINT16
- removed joint JOINT17
- removed joint JOINT18
- removed joint JOINT19
- removed joint JOINT2
- removed joint JOINT20
- removed joint JOINT21
- removed joint JOINT22
- removed joint JOINT23
- removed joint JOINT3
- removed joint JOINT4
- removed joint JOINT5
- removed joint JOINT6
- removed joint JOINT7
- removed joint JOINT8
- removed joint JOINT9
- added joint head-neck-p: type revolute, parent LINK12, child LINK13, origin xyz=-0.000000 -0.018000 0.032500 rpy=1.78188966 -1.57079633 -0.21109333, axis  0  0  1, limit lower=-4.71239000 upper=4.71239000 effort=200.00 velocity=40.00
- added joint head-neck-y: type revolute, parent BASE, child LINK12, origin xyz=0.000000 -0.007250 0.077500 rpy=-0.00000000 0.00000000 -1.57079633, axis  0  0  1, limit lower=-4.71239000 upper=4.71239000 effort=200.00 velocity=40.00
- added joint larm-elbow-p: type revolute, parent LINK2, child LINK3, origin xyz=0.017500 0.000000 0.025500 rpy=0.61547971 1.57079633 0.61547971, axis  0  0  1, limit lower=-4.71239000 upper=4.71239000 effort=200.00 velocity=40.00
- added joint larm-gripper-r: type revolute, parent LINK3, child LINK4, origin xyz=-0.055500 -0.018000 -0.018000 rpy=2.25741790 -1.57079633 -0.68662157, axis  0  0  1, limit lower=-4.71239000 upper=4.71239000 effort=200.00 velocity=40.00
- added joint larm-gripper2-r: type revolute, parent LINK3, child LINK5, origin xyz=-0.066000 -0.018000 -0.039000 rpy=2.25741790 -1.57079633 -0.68662157, axis  0  0  1, limit lower=-4.71239000 upper=4.71239000 effort=200.00 velocity=40.00
- added joint larm-shoulder-p: type revolute, parent BASE, child LINK0, origin xyz=-0.051000 -0.007250 0.059500 rpy=1.57079633 -0.00000000 -1.57079633, axis  0  0  1, limit lower=-4.71239000 upper=4.71239000 effort=200.00 velocity=40.00
- added joint larm-shoulder-r: type revolute, parent LINK0, child LINK1, origin xyz=0.000000 0.017500 0.025500 rpy=0.34877100 1.57079633 1.91956733, axis  0  0  1, limit lower=-4.71239000 upper=4.71239000 effort=200.00 velocity=40.00
- added joint larm-shoulder-y: type revolute, parent LINK1, child LINK2, origin xyz=-0.070000 -0.000000 -0.018000 rpy=-1.57079633 -0.00000000 1.57079633, axis  0  0  1, limit lower=-4.71239000 upper=4.71239000 effort=200.00 velocity=40.00
- added joint lleg-ankle-p: type revolute, parent LINK21, child LINK22, origin xyz=-0.023500 -0.053000 -0.035500 rpy=-3.14159265 0.00000000 -1.57079633, axis  0  0  1, limit lower=-4.71239000 upper=4.71239000 effort=200.00 velocity=40.00
- added joint lleg-ankle-r: type revolute, parent LINK22, child LINK23, origin xyz=0.000000 -0.017000 -0.018000 rpy=-1.57079633 -0.00000000 0.00000000, axis  0  0  1, limit lower=-4.71239000 upper=4.71239000 effort=200.00 velocity=40.00
- added joint lleg-crotch-p: type revolute, parent LINK19, child LINK20, origin xyz=0.000000 -0.018000 0.017000 rpy=1.57079633 0.00000000 0.00000000, axis  0  0  1, limit lower=-4.71239000 upper=4.71239000 effort=200.00 velocity=40.00
- added joint lleg-crotch-r: type revolute, parent BASE, child LINK19, origin xyz=-0.023500 -0.017000 -0.036000 rpy=-1.29249667 -1.57079633 -0.27829966, axis  0  0  1, limit lower=-4.71239000 upper=4.71239000 effort=200.00 velocity=40.00
- added joint lleg-knee-p: type revolute, parent LINK20, child LINK21, origin xyz=-0.058000 -0.000000 -0.000000 rpy=-0.00000000 -0.00000000 0.00000000, axis  0  0  1, limit lower=-4.71239000 upper=4.71239000 effort=200.00 velocity=40.00
- added joint rarm-elbow-p: type revolute, parent LINK8, child LINK9, origin xyz=0.017500 0.000000 0.025500 rpy=-0.20903330 1.57079633 -0.20903330, axis  0  0  1, limit lower=-4.71239000 upper=4.71239000 effort=200.00 velocity=40.00
- added joint rarm-gripper-r: type revolute, parent LINK9, child LINK10, origin xyz=-0.055500 -0.018000 -0.018000 rpy=2.27590767 -1.57079633 -0.70511135, axis  0  0  1, limit lower=-4.71239000 upper=4.71239000 effort=200.00 velocity=40.00
- added joint rarm-gripper2-r: type revolute, parent LINK9, child LINK11, origin xyz=-0.066000 -0.018000 -0.039000 rpy=2.27590767 -1.57079633 -0.70511135, axis  0  0  1, limit lower=-4.71239000 upper=4.71239000 effort=200.00 velocity=40.00
- added joint rarm-shoulder-p: type revolute, parent BASE, child LINK6, origin xyz=0.051000 -0.007250 0.059500 rpy=-1.57079633 0.00000000 -1.57079633, axis  0  0  1, limit lower=-4.71239000 upper=4.71239000 effort=200.00 velocity=40.00
- added joint rarm-shoulder-r: type revolute, parent LINK6, child LINK7, origin xyz=0.000000 0.017500 0.025500 rpy=-0.46364761 1.57079633 1.10714872, axis  0  0  1, limit lower=-4.71239000 upper=4.71239000 effort=200.00 velocity=40.00
- added joint rarm-shoulder-y: type revolute, parent LINK7, child LINK8, origin xyz=-0.070000 -0.000000 -0.018000 rpy=-1.57079633 -0.00000000 1.57079633, axis  0  0  1, limit lower=-4.71239000 upper=4.71239000 effort=200.00 velocity=40.00
- added joint rleg-ankle-p: type revolute, parent LINK16, child LINK17, origin xyz=-0.023500 -0.053000 -0.035500 rpy=-3.14159265 0.00000000 -1.57079633, axis  0  0  1, limit lower=-4.71239000 upper=4.71239000 effort=200.00 velocity=40.00
- added joint rleg-ankle-r: type revolute, parent LINK17, child LINK18, origin xyz=0.000000 -0.017000 -0.018000 rpy=-1.57079633 -0.00000000 0.00000000, axis  0  0  1, limit lower=-4.71239000 upper=4.71239000 effort=200.00 velocity=40.00
- added joint rleg-crotch-p: type revolute, parent LINK14, child LINK15, origin xyz=0.000000 -0.018000 0.017000 rpy=1.57079633 0.00000000 0.00000000, axis  0  0  1, limit lower=-4.71239000 upper=4.71239000 effort=200.00 velocity=40.00
- added joint rleg-crotch-r: type revolute, parent BASE, child LINK14, origin xyz=0.023500 -0.017000 -0.036000 rpy=-1.29249667 -1.57079633 -0.27829966, axis  0  0  1, limit lower=-4.71239000 upper=4.71239000 effort=200.00 velocity=40.00
- added joint rleg-knee-p: type revolute, parent LINK15, child LINK16, origin xyz=-0.058000 -0.000000 -0.000000 rpy=-0.00000000 -0.00000000 0.00000000, axis  0  0  1, limit lower=-4.71239000 upper=4.71239000 effort=200.00 velocity=40.00
