Commit message: [user] update

File: sample/kxr_auv/larm.urdf (robot description, URDF)
Before this commit: robot larm, 6 links, 5 joints
Links:
- link BASE: mass 0.011949 -> 0.003379; geometry collision box size=0.004400 0.001200 0.000800; collision box size=0.004400 0.007600 0.002400
Joints:
- joint larm-elbow-p: origin xyz=0.017500 -0.000000 0.025500 rpy=0.81482692 1.57079633 0.81482692 -> xyz=0.017500 0.000000 0.025500 rpy=0.81482692 1.57079633 0.81482692
- joint larm-shoulder-r: origin xyz=0.017500 0.000000 0.023000 rpy=0.00000000 1.57079633 0.00000000 -> xyz=0.004500 0.000000 0.023000 rpy=0.00000000 1.57079633 0.00000000

File: sample/kxr_auv/rarm.urdf (robot description, URDF)
Before this commit: robot rarm, 6 links, 5 joints
Links:
- link BASE: mass 0.011949 -> 0.003379; geometry collision box size=0.004400 0.001200 0.000800; collision box size=0.004400 0.007600 0.002400
Joints:
- joint rarm-elbow-p: origin xyz=0.017500 -0.000000 0.025500 rpy=0.81482692 1.57079633 0.81482692 -> xyz=0.017500 0.000000 0.025500 rpy=0.81482692 1.57079633 0.81482692
- joint rarm-shoulder-r: origin xyz=0.017500 0.000000 0.023000 rpy=0.00000000 1.57079633 0.00000000 -> xyz=0.004500 0.000000 0.023000 rpy=0.00000000 1.57079633 0.00000000
