Commit message: [user] update

File: sample/kxr_auv/torso.urdf (robot description, URDF)
Before this commit: robot torso, 3 links, 2 joints
Joints:
- removed joint JOINT1
- added joint head-neck-p: type revolute, parent LINK0, child LINK1, origin xyz=-0.010500 -0.018000 0.032500 rpy=1.42371797 -1.57079633 0.14707836, axis  0  0  1, limit lower=-4.71239000 upper=4.71239000 effort=200.00 velocity=40.00

Commit message: [user] update

File: sample/kxr_auv/torso.urdf (robot description, URDF)
Before this commit: robot torso, 3 links, 2 joints
Joints:
- removed joint JOINT0
- added joint head-neck-y: type revolute, parent BASE, child LINK0, origin xyz=0.000000 -0.007250 0.077500 rpy=-0.00000000 0.00000000 -1.57079633, axis  0  0  1, limit lower=-4.71239000 upper=4.71239000 effort=200.00 velocity=40.00

Commit message: [user] update torso

File: sample/kxr_auv/torso.urdf (robot description, URDF)
Before this commit: robot torso, 3 links, 2 joints
Links:
- added link LINK2, mass 0.03619; collision box size=0.002000 0.003600 0.002400; collision box size=0.002000 0.004400 0.000400
- added link LINK3, mass 0.325949; collision box size=0.004400 0.001200 0.000800; collision box size=0.004400 0.001200 0.000800
- link LINK0: mass 0.03619 -> 0.00857; geometry collision box size=0.004400 0.001200 0.000800; collision box size=0.004400 0.007600 0.002000
- link LINK1: mass 0.325949 -> 0.00857; geometry collision box size=0.004400 0.001200 0.000800; collision box size=0.004400 0.007600 0.002000
Joints:
- added joint larm-shoulder-p: type revolute, parent BASE, child LINK0, origin xyz=-0.051000 -0.007250 0.059500 rpy=1.57079633 -0.00000000 -1.57079633, axis  0  0  1, limit lower=-4.71239000 upper=4.71239000 effort=200.00 velocity=40.00
- added joint rarm-shoulder-p: type revolute, parent BASE, child LINK1, origin xyz=0.051000 -0.007250 0.059500 rpy=-1.57079633 0.00000000 -1.57079633, axis  0  0  1, limit lower=-4.71239000 upper=4.71239000 effort=200.00 velocity=40.00
- joint head-neck-p: child LINK1 -> LINK3; parent LINK0 -> LINK2
- joint head-neck-y: child LINK0 -> LINK2
