Commit message: [user] update test roboasm

File: sample/kxr_auv/test.urdf (robot description, URDF)
Before this commit: robot test, 2 links, 1 joints
Joints:
- removed joint JOINT0
- added joint hoge: type revolute, parent BASE, child LINK0, origin xyz=0.000000 0.000000 0.018000 rpy=0.00000000 -0.00000000 3.14159265, axis  0  0  1, limit lower=-4.71239000 upper=4.71239000 effort=200.00 velocity=40.00
