Commit message: [user] add camera model

File: sample/kxr_auv/kxr_auv_fullbody_initial.urdf (robot description, URDF)
Before this commit: robot kxr_auv_fullbody_initial, 25 links, 24 joints
Links:
- added link camera00_optical
Joints:
- added joint camera00_fixed_joint: type fixed, parent LINK13, child camera00_optical, origin xyz=0.050000000000 0.009500000000 -0.070200000000 rpy=1.570796326795 0.000000000000 -1.570796326795

Commit message: [user] update camera position

File: sample/kxr_auv/kxr_auv_fullbody_initial.urdf (robot description, URDF)
Before this commit: robot kxr_auv_fullbody_initial, 26 links, 25 joints
Joints:
- joint camera00_fixed_joint: origin xyz=0.050000000000 0.009500000000 -0.070200000000 rpy=1.570796326795 0.000000000000 -1.570796326795 -> xyz=0.044000000000 0.007000000000 -0.017500000000 rpy=1.570796326795 -0.000000000000 -3.141592653590

Commit message: [user] update initial

File: sample/kxr_auv/kxr_auv_fullbody_initial.urdf (robot description, URDF)
Before this commit: robot kxr_auv_fullbody_initial, 26 links, 25 joints
Joints:
- joint head-neck-p: origin xyz=-0.010500 -0.018000 0.032500 rpy=1.42371797 -1.57079633 0.14707836 -> xyz=-0.010500 -0.018000 0.032500 rpy=1.34156439 -1.57079633 0.22923193
- joint larm-elbow-p: origin xyz=0.017500 -0.000000 0.025500 rpy=0.08485739 1.57079633 0.08485739 -> xyz=0.017500 -0.000000 0.025500 rpy=1.04133636 1.57079633 1.04133636
- joint larm-gripper-r: origin xyz=-0.055500 -0.018000 -0.018000 rpy=2.08202704 -1.57079633 -0.51123071 -> xyz=-0.055500 -0.018000 -0.018000 rpy=2.04519621 -1.57079633 -0.47439988
- joint larm-gripper2-r: origin xyz=-0.066000 -0.018000 -0.039000 rpy=2.08202704 -1.57079633 -0.51123071 -> xyz=-0.066000 -0.018000 -0.039000 rpy=2.04519621 -1.57079633 -0.47439988
- joint larm-shoulder-r: origin xyz=-0.012374 0.012374 0.025500 rpy=1.11649424 1.57079633 -2.81049658 -> xyz=-0.012374 0.012374 0.025500 rpy=0.69865982 1.57079633 3.05485431
- joint lleg-crotch-r: origin xyz=-0.023500 -0.017000 -0.036000 rpy=-1.29249667 -1.57079633 -0.27829966 -> xyz=-0.023500 -0.017000 -0.036000 rpy=-1.34608516 -1.57079633 -0.22471117
- joint rarm-elbow-p: origin xyz=0.017500 0.000000 0.025500 rpy=0.66772715 1.57079633 0.66772715 -> xyz=0.017500 -0.000000 0.025500 rpy=1.20268268 1.57079633 1.20268268
- joint rarm-gripper-r: origin xyz=-0.055500 -0.018000 -0.018000 rpy=2.38743432 -1.57079633 -0.81663800 -> xyz=-0.055500 -0.018000 -0.018000 rpy=2.16797298 -1.57079633 -0.59717666
- joint rarm-gripper2-r: origin xyz=-0.066000 -0.018000 -0.039000 rpy=2.38743432 -1.57079633 -0.81663800 -> xyz=-0.066000 -0.018000 -0.039000 rpy=2.16797298 -1.57079633 -0.59717666
- joint rarm-shoulder-r: origin xyz=0.012374 0.012374 0.025500 rpy=1.02344453 1.57079633 1.80884269 -> xyz=0.012374 0.012374 0.025500 rpy=1.37669023 1.57079633 2.16208839
- joint rleg-crotch-r: origin xyz=0.023500 -0.017000 -0.036000 rpy=-1.29249667 -1.57079633 -0.27829966 -> xyz=0.023500 -0.017000 -0.036000 rpy=-1.34608516 -1.57079633 -0.22471117

Commit message: [user] update model

File: sample/kxr_auv/kxr_auv_fullbody_initial.urdf (robot description, URDF)
Before this commit: robot kxr_auv_fullbody_initial, 26 links, 25 joints
Joints:
- joint head-neck-p: origin xyz=-0.010500 -0.018000 0.032500 rpy=1.34156439 -1.57079633 0.22923193 -> xyz=-0.010500 -0.018000 0.032500 rpy=1.57079633 -1.57079633 0.00000000
- joint head-neck-y: origin xyz=0.000000 -0.007250 0.077500 rpy=-0.00000000 0.00000000 -1.57079633 -> xyz=0.000000 -0.007250 0.077500 rpy=-0.00000000 -0.00000000 -1.57079633
- joint larm-elbow-p: origin xyz=0.017500 -0.000000 0.025500 rpy=1.04133636 1.57079633 1.04133636 -> xyz=0.017500 -0.000000 0.025500 rpy=0.55897139 1.57079633 0.55897139
- joint larm-gripper-r: origin xyz=-0.055500 -0.018000 -0.018000 rpy=2.04519621 -1.57079633 -0.47439988 -> xyz=-0.055500 -0.018000 -0.018000 rpy=2.24553727 -1.57079633 -0.67474094
- joint larm-gripper2-r: origin xyz=-0.066000 -0.018000 -0.039000 rpy=2.04519621 -1.57079633 -0.47439988 -> xyz=-0.066000 -0.018000 -0.039000 rpy=2.24553727 -1.57079633 -0.67474094
- joint larm-shoulder-r: origin xyz=-0.012374 0.012374 0.025500 rpy=0.69865982 1.57079633 3.05485431 -> xyz=-0.012374 0.012374 0.025500 rpy=1.23755203 1.57079633 -2.68943879
- joint lleg-crotch-r: origin xyz=-0.023500 -0.017000 -0.036000 rpy=-1.34608516 -1.57079633 -0.22471117 -> xyz=-0.023500 -0.017000 -0.036000 rpy=-1.36775111 -1.57079633 -0.20304522
- joint rarm-elbow-p: origin xyz=0.017500 -0.000000 0.025500 rpy=1.20268268 1.57079633 1.20268268 -> xyz=0.017500 0.000000 0.025500 rpy=-0.39121759 1.57079633 -0.39121759
- joint rarm-gripper-r: origin xyz=-0.055500 -0.018000 -0.018000 rpy=2.16797298 -1.57079633 -0.59717666 -> xyz=-0.055500 -0.018000 -0.018000 rpy=2.24131788 -1.57079633 -0.67052156
- joint rarm-gripper2-r: origin xyz=-0.066000 -0.018000 -0.039000 rpy=2.16797298 -1.57079633 -0.59717666 -> xyz=-0.066000 -0.018000 -0.039000 rpy=2.24131788 -1.57079633 -0.67052156
- joint rarm-shoulder-r: origin xyz=0.012374 0.012374 0.025500 rpy=1.37669023 1.57079633 2.16208839 -> xyz=0.012374 0.012374 0.025500 rpy=0.96470161 1.57079633 1.75009977
- joint rleg-crotch-r: origin xyz=0.023500 -0.017000 -0.036000 rpy=-1.34608516 -1.57079633 -0.22471117 -> xyz=0.023500 -0.017000 -0.036000 rpy=-1.36775111 -1.57079633 -0.20304522

Commit message: [student_projects] update model

File: sample/kxr_auv/kxr_auv_fullbody_initial.urdf (robot description, URDF)
Before this commit: robot kxr_auv_fullbody_initial, 26 links, 25 joints
Joints:
- joint head-neck-p: origin xyz=-0.010500 -0.018000 0.032500 rpy=1.57079633 -1.57079633 0.00000000 -> xyz=-0.010500 -0.018000 0.032500 rpy=1.34156439 -1.57079633 0.22923193
- joint head-neck-y: origin xyz=0.000000 -0.007250 0.077500 rpy=-0.00000000 -0.00000000 -1.57079633 -> xyz=0.000000 -0.007250 0.077500 rpy=-0.00000000 0.00000000 -1.57079633
- joint larm-elbow-p: origin xyz=0.017500 -0.000000 0.025500 rpy=0.55897139 1.57079633 0.55897139 -> xyz=0.017500 -0.000000 0.025500 rpy=1.04133636 1.57079633 1.04133636
- joint larm-gripper-r: origin xyz=-0.055500 -0.018000 -0.018000 rpy=2.24553727 -1.57079633 -0.67474094 -> xyz=-0.055500 -0.018000 -0.018000 rpy=2.04519621 -1.57079633 -0.47439988
- joint larm-gripper2-r: origin xyz=-0.066000 -0.018000 -0.039000 rpy=2.24553727 -1.57079633 -0.67474094 -> xyz=-0.066000 -0.018000 -0.039000 rpy=2.04519621 -1.57079633 -0.47439988
- joint larm-shoulder-r: origin xyz=-0.012374 0.012374 0.025500 rpy=1.23755203 1.57079633 -2.68943879 -> xyz=-0.012374 0.012374 0.025500 rpy=0.69865982 1.57079633 3.05485431
- joint lleg-crotch-r: origin xyz=-0.023500 -0.017000 -0.036000 rpy=-1.36775111 -1.57079633 -0.20304522 -> xyz=-0.023500 -0.017000 -0.036000 rpy=-1.34608516 -1.57079633 -0.22471117
- joint rarm-elbow-p: origin xyz=0.017500 0.000000 0.025500 rpy=-0.39121759 1.57079633 -0.39121759 -> xyz=0.017500 -0.000000 0.025500 rpy=1.20268268 1.57079633 1.20268268
- joint rarm-gripper-r: origin xyz=-0.055500 -0.018000 -0.018000 rpy=2.24131788 -1.57079633 -0.67052156 -> xyz=-0.055500 -0.018000 -0.018000 rpy=2.16797298 -1.57079633 -0.59717666
- joint rarm-gripper2-r: origin xyz=-0.066000 -0.018000 -0.039000 rpy=2.24131788 -1.57079633 -0.67052156 -> xyz=-0.066000 -0.018000 -0.039000 rpy=2.16797298 -1.57079633 -0.59717666
- joint rarm-shoulder-r: origin xyz=0.012374 0.012374 0.025500 rpy=0.96470161 1.57079633 1.75009977 -> xyz=0.012374 0.012374 0.025500 rpy=1.37669023 1.57079633 2.16208839
- joint rleg-crotch-r: origin xyz=0.023500 -0.017000 -0.036000 rpy=-1.36775111 -1.57079633 -0.20304522 -> xyz=0.023500 -0.017000 -0.036000 rpy=-1.34608516 -1.57079633 -0.22471117
